File: pcb/smartwatch_soc.kicad_pcb (KiCad board)
At the start: 2 copper layers, 25.4 x 38.1 mm, 33 parts, among them J1 Battery Socket, J2 USB_A, Q1 PN2222A, Q2 PN2222A, SW1 EN_Switch, SW2 Button, SW3 Button, SW4 Button, SW5 Button, U1 ESP32-S3-MINI-1U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

Commit message: reset pcb designs
Parts:
- removed C1: 5uF, Capacitor_THT:C_Disc_D3.0mm_W1.6mm_P2.50mm
- removed C2: 1uF, Capacitor_THT:C_Disc_D3.0mm_W1.6mm_P2.50mm
- removed U4: MCP1727-3302xMF, Package_DFN_QFN:DFN-8-1EP_3x3mm_P0.65mm_EP1.55x2.4mm
- added C3: 4.7uF, Capacitor_THT:C_Disc_D3.0mm_W1.6mm_P2.50mm, F.Cu at (93.9, 36.0)
- added C4: 0.1uF, Capacitor_THT:C_Disc_D3.0mm_W1.6mm_P2.50mm, F.Cu at (93.9, 39.2)
- added D5: 1N5820, Diode_THT:D_DO-201AD_P15.24mm_Horizontal, F.Cu at (66.8, 32.0)
- added D7: 1N5820, Diode_THT:D_DO-201AD_P15.24mm_Horizontal, F.Cu at (66.8, 38.8)
- added Q3: PN2222A, Package_TO_SOT_THT:TO-92_Inline, F.Cu at (84.6, 57.0)
- added R14: 1kR, Resistor_THT:R_Axial_DIN0204_L3.6mm_D1.6mm_P2.54mm_Vertical, F.Cu at (77.2, 70.7)
- added R15: R, Resistor_THT:R_Axial_DIN0204_L3.6mm_D1.6mm_P2.54mm_Vertical, F.Cu at (77.2, 73.8)
- D2, D3, D4: footprint LED_SMD:LED_0201_0603Metric -> LED_THT:LED_D2.0mm_W4.0mm_H2.8mm_FlatTop
- J1: moved to F.Cu
- R1, R10, R11, R12, R13, R2, R3, R4, R5, R6, R7, R8, R9: footprint Resistor_SMD:R_0201_0603Metric -> Resistor_THT:R_Axial_DIN0204_L3.6mm_D1.6mm_P2.54mm_Vertical
- moved SW2 44.6 mm to (61.1, 31.1)
- moved SW5 44.6 mm to (61.1, 47.3)
- moved SW4 44.6 mm to (61.1, 41.9)
- moved SW3 44.6 mm to (61.1, 36.5)
- moved U2 43.6 mm to (60.5, 57.8), turned to 0 degrees
- moved D3 41.3 mm to (90.8, 48.9)
- moved D4 38.9 mm to (90.8, 53.3)
- moved J1 36.7 mm to (87.4, 37.2), turned to 0 degrees
- moved Q1 35.3 mm to (84.6, 45.4)
- moved Q2 35.3 mm to (84.6, 51.2)
- moved R11 29.0 mm to (77.2, 61.2)
- moved R6 28.3 mm to (71.6, 61.2)
- moved R12 27.7 mm to (77.2, 64.4)
- moved R7 27.0 mm to (71.6, 64.4)
- moved R13 26.3 mm to (77.2, 67.5)
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Connections:
- D1 pad 2: VBUS_5V -> Net-(D5-K)
- J2 pad 1: VBUS_5V -> Net-(D5-A)
- R1 pad 1: VBUS_5V -> Net-(D5-K)
- SW1 pad 1: Battery_3.3V -> 3.3V
- U5 pad 6: unconnected-(U5-VDD-Pad6) -> 3.3V
- U5 pad 7: VBUS_5V -> Net-(D5-K)
- U5 pad 9: unconnected-(U5-~{RST}-Pad9) -> Net-(U5-~{RST})
Routing:
- net GND: track 157.7 -> 0.00 mm
- net ESP_3V3: track 55.1 -> 0.00 mm
- net Battery_3.3V: track 32.4 -> 0.00 mm
- net GPIO34: track 17.7 -> 0.00 mm
- net GPIO48: track 17.2 -> 0.00 mm
- net GPIO18: track 16.4 -> 0.00 mm
- net GPIO17: track 14.4 -> 0.00 mm
- net GPIO16: track 12.6 -> 0.00 mm
- net Net-(D7-A): track 12.1 -> 0.00 mm
Other:
- board outline removed
