File: pcb/smartwatch_soc.kicad_pcb (KiCad board)
At the start: 2 copper layers, 37 parts, among them J1 Battery Socket, J2 USB_A, Q1 PN2222A, Q2 PN2222A, Q3 PN2222A, SW1 EN_Switch, SW2 Button, SW3 Button, SW4 Button, SW5 Button, U1 ESP32-S3-MINI-1U, U2 LSM6DS3, U3 OLED_Display, U5 CP2102N-Axx-xQFN20

Commit message: added footprints
Parts:
- removed C3: 4.7uF, Capacitor_THT:C_Disc_D3.0mm_W1.6mm_P2.50mm
- removed C4: 0.1uF, Capacitor_THT:C_Disc_D3.0mm_W1.6mm_P2.50mm
- removed D1: SP0503BAHT, Package_TO_SOT_SMD:SOT-143
- removed D2, D3, D4: LED, LED_THT:LED_D2.0mm_W4.0mm_H2.8mm_FlatTop
- removed D5, D7: 1N5820, Diode_THT:D_DO-201AD_P15.24mm_Horizontal
- removed J1: Battery Socket, Connector_JST:JST_PH_B2B-PH-K_1x02_P2.00mm_Vertical
- removed J2: USB_A, Connector_USB:USB_A_TE_292303-7_Horizontal
- removed Q1, Q2, Q3: PN2222A, Package_TO_SOT_THT:TO-92_Inline
- removed R1: 22.1kR, Resistor_THT:R_Axial_DIN0204_L3.6mm_D1.6mm_P2.54mm_Vertical
- removed R10, R15, R6, R7, R9: R, Resistor_THT:R_Axial_DIN0204_L3.6mm_D1.6mm_P2.54mm_Vertical
- removed R11, R8: 500R, Resistor_THT:R_Axial_DIN0204_L3.6mm_D1.6mm_P2.54mm_Vertical
- removed R12, R13, R3, R4, R5: 10kR, Resistor_THT:R_Axial_DIN0204_L3.6mm_D1.6mm_P2.54mm_Vertical
- removed R14: 1kR, Resistor_THT:R_Axial_DIN0204_L3.6mm_D1.6mm_P2.54mm_Vertical
- removed R2: 47.5kR, Resistor_THT:R_Axial_DIN0204_L3.6mm_D1.6mm_P2.54mm_Vertical
- removed SW1: EN_Switch, Button_Switch_SMD:SW_DIP_SPSTx01_Slide_6.7x4.1mm_W6.73mm_P2.54mm_LowProfile_JPin
- removed SW2, SW3, SW4, SW5: Button, Button_Switch_SMD:SW_SPST_CK_KMS2xxGP
- removed U1: ESP32-S3-MINI-1U, RF_Module:ESP32-S2-MINI-1U
- removed U2: LSM6DS3, Package_LGA:LGA-14_3x2.5mm_P0.5mm_LayoutBorder3x4y
- removed U3: OLED_Display, Connector_PinHeader_1.00mm:PinHeader_1x04_P1.00mm_Vertical
- removed U5: CP2102N-Axx-xQFN20, Package_DFN_QFN:SiliconLabs_QFN-20-1EP_3x3mm_P0.5mm_EP1.8x1.8mm

Commit message: started pcb layout
Parts:
- added C1: 100nF, Capacitor_THT:C_Disc_D5.0mm_W2.5mm_P2.50mm, F.Cu at (146.1, 82.0)
- added C2: 100nF, Capacitor_THT:C_Disc_D5.0mm_W2.5mm_P2.50mm, F.Cu at (149.2, 84.5)
- added C3: 470pF, Capacitor_THT:C_Disc_D5.0mm_W2.5mm_P2.50mm, F.Cu at (155.5, 82.5)
- added C4: 2.2uF, Capacitor_THT:C_Disc_D5.0mm_W2.5mm_P2.50mm, F.Cu at (158.0, 85.6)
- added C5: 0.1uF, Capacitor_THT:C_Disc_D5.0mm_W2.5mm_P2.50mm, F.Cu at (174.0, 63.5)
- added C6: 22uF, Capacitor_THT:C_Disc_D5.0mm_W2.5mm_P2.50mm, F.Cu at (148.6, 63.5)
- added C7: 0.1uF, Capacitor_THT:C_Disc_D5.0mm_W2.5mm_P2.50mm, F.Cu at (151.1, 66.7)
- added C8: 0.1uF, Capacitor_THT:C_Disc_D5.0mm_W2.5mm_P2.50mm, F.Cu at (151.1, 72.4)
- added C9: 1uF, Capacitor_THT:C_Disc_D5.0mm_W2.5mm_P2.50mm, F.Cu at (174.0, 66.7)
- added D1: LED_3V3, LED_THT:LED_D1.8mm_W3.3mm_H2.4mm, F.Cu at (177.8, 92.1)
- added D10: 1N5819, Diode_THT:D_DO-41_SOD81_P10.16mm_Horizontal, F.Cu at (166.6, 78.0)
- added D6: ESD9B3.3ST5G, Diode_SMD:D_SOD-923, F.Cu at (164.1, 88.2)
- added D8: ESD9B3.3ST5G, Diode_SMD:D_SOD-923, F.Cu at (161.6, 88.2)
- added D9: ESD9B3.3ST5G, Diode_SMD:D_SOD-923, F.Cu at (162.8, 88.2)
- added J2: USB_B_Micro, Connector_USB:USB_Micro-B_Amphenol_10118194-0001LF_Horizontal, F.Cu at (160.0, 93.9)
- added R12: 10kR, Resistor_THT:R_Axial_DIN0204_L3.6mm_D1.6mm_P5.08mm_Horizontal, F.Cu at (181.4, 71.8)
- added R13: 10kR, Resistor_THT:R_Axial_DIN0204_L3.6mm_D1.6mm_P5.08mm_Horizontal, F.Cu at (172.1, 71.8)
- added R16: 10kR, Resistor_THT:R_Axial_DIN0204_L3.6mm_D1.6mm_P5.08mm_Horizontal, F.Cu at (177.2, 62.9)
- added R18: 5.1kR, Resistor_THT:R_Axial_DIN0204_L3.6mm_D1.6mm_P5.08mm_Horizontal, F.Cu at (176.5, 88.9)
- added R4: 10kR, Resistor_THT:R_Axial_DIN0204_L3.6mm_D1.6mm_P5.08mm_Horizontal, F.Cu at (181.6, 80.6)
- added R5: 10kR, Resistor_THT:R_Axial_DIN0204_L3.6mm_D1.6mm_P5.08mm_Horizontal, F.Cu at (172.1, 80.6)
- added SW1: CK_KMS2xxGP, Button_Switch_SMD:SW_SPST_CK_KMS2xxGP, F.Cu at (146.5, 70.3)
- added SW2: Button, Button_Switch_SMD:SW_SPST_CK_KMS2xxGP, F.Cu at (185.9, 82.4)
- added SW3: Button, Button_Switch_SMD:SW_SPST_CK_KMS2xxGP, F.Cu at (176.4, 82.4)
- added SW4: Button, Button_Switch_SMD:SW_SPST_CK_KMS2xxGP, F.Cu at (185.7, 73.5)
- added SW5: Button, Button_Switch_SMD:SW_SPST_CK_KMS2xxGP, F.Cu at (176.5, 73.2)
- added SW7: CK_KMS2xxGP, Button_Switch_SMD:SW_SPST_CK_KMS2xxGP, F.Cu at (181.5, 63.7)
- added U1: MIC5219-3.3YM5, Package_TO_SOT_SMD:SOT-23-5, F.Cu at (161.7, 84.0)
- added U2: LSM6DS3, Package_LGA:LGA-14_3x2.5mm_P0.5mm_LayoutBorder3x4y, F.Cu at (147.3, 78.1)
- added U3: OLED_Display, Connector_PinHeader_1.00mm:PinHeader_1x04_P1.00mm_Vertical, F.Cu at (140.3, 81.6)
- added U5: ESP32-S3-MINI-1, RF_Module:ESP32-S2-MINI-1, F.Cu at (161.3, 66.1)
Routing:
- net USB_DP: track 0.00 -> 14.3 mm
- net VBUS: track 0.00 -> 11.7 mm
- net USB_DN: track 0.00 -> 10.9 mm
